File: hardware/garden/garden.sch (KiCad schematic (older format))
At the start: 53 parts, among them J1 CONN_01X40, J2 CONN_01X08, J3 CONN_01X06, J4 CONN_01X10, J5 CONN_01X08, J7 Micro_SD_Card_CD, J8 CONN_01X13, J9 CONN_01X06, M1 ESP-11, M2 CONN_01X01, M3 CONN_01X01, M4 CONN_01X01, M5 CONN_01X01, P1 USB_OTG, Q1 Q_NMOS_GSD, SW1 RESET, SW2 BOOT, U1 AZ1117-3.3, U2 STM32F745ZETx, U3 IS42S16160G, Y1 12MHz

Commit message: Designed garden controller
Parts:
- removed C16: 10uF, Capacitors_SMD:C_0805, symbol ostrich-rescue:C-device
- removed J1: CONN_01X40, ER-CON40HB-2:ER-CON40HB-2, symbol conn1:CONN_01X40
- removed J2, J5: CONN_01X08, Pin_Headers:Pin_Header_Straight_1x08_Pitch2.54mm, symbol conn1:CONN_01X08
- removed J3: CONN_01X06, Pin_Headers:Pin_Header_Straight_1x06_Pitch2.54mm, symbol conn1:CONN_01X06
- removed J4: CONN_01X10, Connector_PinHeader_2.54mm:PinHeader_1x10_P2.54mm_Vertical, symbol conn1:CONN_01X10
- removed J7: Micro_SD_Card_CD, Amphenol:Amphenol_1140084168, symbol micro_sd_card_cd:Micro_SD_Card_CD
- removed J8: CONN_01X13, Pin_Headers:Pin_Header_Straight_1x13_Pitch2.54mm, symbol conn1:CONN_01X13
- removed R1, R4, R5, R6: 10KR, Resistors_SMD:R_0805, symbol ostrich-rescue:R-device
- removed U3: IS42S16160G, TSOPII:TSOPII-54_10.16x22.22mm-Pitch0.8mm, symbol is42s16160g:IS42S16160G
- added C16, C18, C19, C20: 0.1uF, Capacitor_SMD:C_0805_2012Metric_Pad1.15x1.40mm_HandSolder, symbol Device:C
- added C17: 1uF, Capacitor_SMD:C_0805_2012Metric_Pad1.15x1.40mm_HandSolder, symbol Device:C
- added C21, C22: 220uF, Capacitor_THT:CP_Radial_D8.0mm_P3.50mm, symbol Device:CP
- added C23: 22uF, Capacitor_THT:CP_Radial_D6.3mm_P2.50mm, symbol Device:CP
- added D7: D_Schottky, Diode_SMD:D_1206_3216Metric_Pad1.42x1.75mm_HandSolder, symbol ostrich-rescue:D_Schottky-device
- added J1, J3: CONN_01X04, Connector_JST:JST_PH_B4B-PH-SM4-TB_1x04-1MP_P2.00mm_Vertical, symbol conn1:CONN_01X04
- added J10: CONN_01X10, Connector_PinHeader_2.54mm:PinHeader_1x10_P2.54mm_Vertical, symbol conn1:CONN_01X10
- added J2, J4, J5, J6: CONN_01X02, TerminalBlock_Phoenix:TerminalBlock_Phoenix_MKDS-3-2-5.08_1x02_P5.08mm_Horizontal, symbol conn1:CONN_01X02
- added J7, J8: CONN_01X04, TerminalBlock_Phoenix:TerminalBlock_Phoenix_MPT-0,5-4-2.54_1x04_P2.54mm_Horizontal, symbol conn1:CONN_01X04
- added Q2, Q3: Q_NMOS_GDS, Package_TO_SOT_THT:TO-220-3_Vertical, symbol Device:Q_NMOS_GDS
- added R1, R4: 10mR, Resistor_SMD:R_1206_3216Metric_Pad1.42x1.75mm_HandSolder, symbol Device:R
- added R11, R12, R5: 1kR, Resistor_SMD:R_0805_2012Metric_Pad1.15x1.40mm_HandSolder, symbol Device:R
- added R6: 6.8R, Resistor_SMD:R_0805_2012Metric_Pad1.15x1.40mm_HandSolder, symbol Device:R
- added U3: R-78B5.0-2.0, Converter_DCDC:Converter_DCDC_RECOM_R-78B-2.0_THT, symbol Regulator_Switching:R-78B5.0-2.0
- added U4: MIC4427, Package_SO:SOIC-8_3.9x4.9mm_P1.27mm, symbol Driver_FET:MIC4427
- added U5, U6, U8: INA193, Package_TO_SOT_SMD:SOT-23-5, symbol Amplifier_Current:INA193
- added U7: TEC2-1215WI, Converter_DCDC:Converter_DCDC_TRACO_TMR-xxxx_THT, symbol Converter_DCDC:TEC2-1215WI
- C14: footprint Capacitors_SMD:C_0805 -> Capacitor_SMD:C_0805_2012Metric_Pad1.15x1.40mm_HandSolder
- C15: value 10uF -> 0.1uF; footprint Capacitors_SMD:C_0805 -> Capacitor_SMD:C_0805_2012Metric_Pad1.15x1.40mm_HandSolder
- M2, M3, M4, M5: footprint Mechanical:M2_HOLE -> MountingHole:MountingHole_6.4mm_M6
Connections:
- net labels added: +12V, PF0, PF1, PF2, PRESSURE_CUR, PRESSURE_PWR, SCL, SDA, SW0_CUR, SW0_GATE, SW0_SIG, SW1_CUR, SW1_GATE, SW1_SIG, VD_RX, VD_TX
- net labels removed: A0, A1, A10, A11, A12, A2, A3, A4, A5, A6, A7, A8, A9, BA0, BA1, D0, D1, D10, D11, D12, D13, D14, D15, D2, D3, D4, D5, D6, D7, D8, D9, LCD_BL, LCD_TE, NBL0, NBL1, PA0, PA10, PA15, PA4, PA5, PA7, PA8, PA9, PC10, PC11, PC12, PC6, PC7, PC8, PC9, PD11, PD12, PD13, PG6, PG7, SDCKE0, SDCLK, SDNCAS, SDNE0, SDNRAS, SDNWE, SD_CD, SD_CS, SD_MISO, SD_MOSI, SD_SCLK, TOUCH_INT, TOUCH_RESET, TOUCH_SCL, TOUCH_SDA, TOUCH_WAKE, ~LCD_CS, ~LCD_RD, ~LCD_WR
- wire segments 429 -> 299
- no-connect marks 14 -> 3
Other:
- note added: "Alternative with Tx/Rx reversed"
- note added: "Future Expansion"
- note added: "I2C Sensors"
- note added: "LEDs"
- note added: "M6 mounting holes"
- note added: "Pressure transducer (4-20mA current loop)"
- note added: "SmartSolar VE Direct interface"
- note added: "Solar Power Input"
- note added: "Switched outputs"
- note added: "VD bus is 5V, so we have to use a\n5V tolerant pin for RX"
- note added: "Wifi"
- note removed: "Analog"
- note removed: "Bottom right"
- note removed: "Bottom. Can only be used if LCD isn't used."
- note removed: "BuyDisplay LCD, 8080 16-bit parallel (mirrored)\n+ Capacitive touch"
- note removed: "M2 mounting holes"
- note removed: "Power"
- note removed: "Top right (0.1" aligned)"
- moved on the sheet: C10, C11, C12, C8, C9, D3, D4, D5, D6, R10, R7, R8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

Commit message: Updated garden controller with test points and back emf diodes
Parts:
- added D8, D9: D_Schottky, Diode_SMD:D_1206_3216Metric_Pad1.42x1.75mm_HandSolder, symbol ostrich-rescue:D_Schottky-device
- added TP1, TP2, TP3, TP4, TP5, TP6, TP7, TP8, TP9, TP?: TestPoint, TestPoint:TestPoint_THTPad_D2.0mm_Drill1.0mm, symbol Connector:TestPoint
Connections:
- wire segments 299 -> 333
Other:
- note added: "Regulators"
- note added: "Reset + Bootloader Activation"
- note added: "STM32 decoupling"
- moved on the sheet: C1, C10, C11, C12, C13, C14, C15, C6, C7, C8, C9, D1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

Commit message: Cosmetic changes and added fab files
Parts:
- added TP11, TP12: TestPoint, TestPoint:TestPoint_THTPad_D2.0mm_Drill1.0mm, symbol Connector:TestPoint
- C2, C3: value 16pF -> 27pF
- gave numbers to parts that had none: 1
Changed lines of the file:
@@
 P 1750 5100
 F 0 "C3" H 1775 5200 50  0000 L CNN
-F 1 "16pF" H 1775 5000 50  0000 L CNN
+F 1 "27pF" H 1775 5000 50  0000 L CNN
 F 2 "Capacitors_SMD:C_0805" H 1788 4950 50  0001 C CNN
 F 3 "" H 1750 5100 50  0000 C CNN
@@
 P 1350 5050
 F 0 "C2" H 1375 5150 50  0000 L CNN
-F 1 "16pF" H 1375 4950 50  0000 L CNN
+F 1 "27pF" H 1375 4950 50  0000 L CNN
 F 2 "Capacitors_SMD:C_0805" H 1388 4900 50  0001 C CNN
 F 3 "" H 1350 5050 50  0000 C CNN
@@
 Text Label 2450 8300 2    50   ~ 0
 SDA
-Wire Wire Line
-	2450 8200 2650 8200
-Wire Wire Line
-	2650 8300 2450 8300
 $Comp
 L conn1:CONN_01X10 J10
@@
 	1250 5900 2650 5900
 $Comp
-L Connector:TestPoint TP?
+L Connector:TestPoint TP10
 U 1 1 5CF48512
 P 12800 7300
-F 0 "TP?" H 12858 7418 50  0000 L CNN
+F 0 "TP10" H 12858 7418 50  0000 L CNN
 F 1 "TestPoint" H 12858 7327 50  0000 L CNN
 F 2 "TestPoint:TestPoint_THTPad_D2.0mm_Drill1.0mm" H 13000 7300 50  0001 C CNN
@@
 Wire Wire Line
 	11850 7300 12800 7300
+$Comp
+L Connector:TestPoint TP12
+U 1 1 5CF604E6
+P 1850 8200
+F 0 "TP12" H 1908 8318 50  0000 L CNN
+F 1 "TestPoint" H 1908 8227 50  0000 L CNN
+F 2 "TestPoint:TestPoint_THTPad_D2.0mm_Drill1.0mm" H 2050 8200 50  0001 C CNN
+F 3 "~" H 2050 8200 50  0001 C CNN
+	1    1850 8200
+	1    0    0    -1
+$EndComp
+$Comp
+L Connector:TestPoint TP11
+U 1 1 5CF613B7
+P 1600 8300
+F 0 "TP11" H 1658 8418 50  0000 L CNN
+F 1 "TestPoint" H 1658 8327 50  0000 L CNN
+F 2 "TestPoint:TestPoint_THTPad_D2.0mm_Drill1.0mm" H 1800 8300 50  0001 C CNN
+F 3 "~" H 1800 8300 50  0001 C CNN
+	1    1600 8300
+	1    0    0    -1
+$EndComp
+Wire Wire Line
+	1600 8300 2650 8300
+Wire Wire Line
+	1850 8200 2650 8200
 $EndSCHEMATC
