File: hardware/garden/garden.sch (KiCad schematic (older format))
At the start: 111 parts, among them J1 CONN_01X04, J10 CONN_01X09, J2 CONN_01X02, J3 CONN_01X02, J4 CONN_01X02, J5 CONN_01X02, J6 CONN_01X02, J7 CONN_01X04, J8 CONN_01X04, J9 USB_B_Micro, M2 CONN_01X01, M3 CONN_01X01, M4 CONN_01X01, M5 CONN_01X01, Q1 Q_NPN_BEC, Q2 Q_NMOS_GDS, Q3 Q_NMOS_GDS, Q4 Q_NPN_BEC, Q5 Q_NMOS_GDS, SW1 SW_Push, U1 INA226, U10 DHT11, U11 AZ1117-3.3, U12 MCP1416, U13 MCP1416, U14 MCP1416, U2 INA226, U3 CP2102, U4 ESP32-WROOM-32, U5 INA226, U7 MCP1416, U9 MP2451DT

Commit message: Increased ESP32 bootloading cap to 4.7uF
Parts:
- C6: value 0.1uF -> 4.7uF; LCSC C1525 -> C23733
Changed lines of the file:
@@
 AR Path="/5F220F22" Ref="C6"  Part="1"
 F 0 "C6" H 3115 5146 50  0000 L CNN
-F 1 "0.1uF" H 3115 5055 50  0000 L CNN
+F 1 "4.7uF" H 3115 5055 50  0000 L CNN
 F 2 "Capacitor_SMD:C_0402_1005Metric" H 3038 4950 50  0001 C CNN
 F 3 "~" H 3000 5100 50  0001 C CNN
-F 4 "C1525" H 3000 5100 50  0001 C CNN "LCSC"
+F 4 "C23733" H 3000 5100 50  0001 C CNN "LCSC"
 	1    3000 5100
 	1    0    0    -1

Commit message: Fixed VE.Direct pinout
Connections:
- wire segments 246 -> 247
Changed lines of the file:
@@
 	0    1    1    0
 $EndComp
-Text Label 15700 6300 2    50   ~ 0
+Text Label 15650 6300 2    50   ~ 0
 VD_TX
-Text Label 15700 5850 2    50   ~ 0
+Text Label 16050 5950 2    50   ~ 0
 VD_RX
 Wire Wire Line
-	16150 5950 15800 5950
-Wire Wire Line
 	16150 5750 15950 5750
-Wire Wire Line
-	15700 5850 16150 5850
 Text Notes 15400 5600 0    50   ~ 0
 SmartSolar VE Direct interface
@@
 L Device:R R3
 U 1 1 5F151B44
-P 15800 6100
-F 0 "R3" H 15870 6146 50  0000 L CNN
-F 1 "1kR" H 15870 6055 50  0000 L CNN
-F 2 "Resistor_SMD:R_0402_1005Metric" V 15730 6100 50  0001 C CNN
-F 3 "~" H 15800 6100 50  0001 C CNN
-F 4 "C11702" H 15800 6100 50  0001 C CNN "LCSC"
-	1    15800 6100
+P 15750 6100
+F 0 "R3" H 15820 6146 50  0000 L CNN
+F 1 "1kR" H 15820 6055 50  0000 L CNN
+F 2 "Resistor_SMD:R_0402_1005Metric" V 15680 6100 50  0001 C CNN
+F 3 "~" H 15750 6100 50  0001 C CNN
+F 4 "C11702" H 15750 6100 50  0001 C CNN "LCSC"
+	1    15750 6100
 	1    0    0    -1
 $EndComp
@@
 L Device:R R13
 U 1 1 5F152029
-P 15800 6500
-F 0 "R13" H 15870 6546 50  0000 L CNN
-F 1 "2kR" H 15870 6455 50  0000 L CNN
-F 2 "Resistor_SMD:R_0402_1005Metric" V 15730 6500 50  0001 C CNN
-F 3 "~" H 15800 6500 50  0001 C CNN
-F 4 "C4109" H 15800 6500 50  0001 C CNN "LCSC"
-	1    15800 6500
+P 15750 6500
+F 0 "R13" H 15820 6546 50  0000 L CNN
+F 1 "2kR" H 15820 6455 50  0000 L CNN
+F 2 "Resistor_SMD:R_0402_1005Metric" V 15680 6500 50  0001 C CNN
+F 3 "~" H 15750 6500 50  0001 C CNN
+F 4 "C4109" H 15750 6500 50  0001 C CNN "LCSC"
+	1    15750 6500
 	1    0    0    -1
 $EndComp
 Wire Wire Line
-	15800 6250 15800 6300
+	15750 6250 15750 6300
 Wire Wire Line
-	15700 6300 15800 6300
-Connection ~ 15800 6300
+	15650 6300 15750 6300
+Connection ~ 15750 6300
 Wire Wire Line
-	15800 6300 15800 6350
+	15750 6300 15750 6350
 $Comp
 L power:GND #PWR011
 U 1 1 5F19B8BB
-P 15800 6650
-F 0 "#PWR011" H 15800 6400 50  0001 C CNN
-F 1 "GND" H 15805 6477 50  0000 C CNN
-F 2 "" H 15800 6650 50  0001 C CNN
-F 3 "" H 15800 6650 50  0001 C CNN
-	1    15800 6650
+P 15750 6650
+F 0 "#PWR011" H 15750 6400 50  0001 C CNN
+F 1 "GND" H 15755 6477 50  0000 C CNN
+F 2 "" H 15750 6650 50  0001 C CNN
+F 3 "" H 15750 6650 50  0001 C CNN
+	1    15750 6650
 	1    0    0    -1
 $EndComp
@@
 Wire Wire Line
 	18150 4700 18100 4700
-Text Label 17600 4900 2    50   ~ 0
+Text Label 17400 4900 2    50   ~ 0
 PRESSURE_SW_GATE
 $Comp
@@
 	-1   0    0    1
 $EndComp
+Wire Wire Line
+	16050 5950 16150 5950
+Wire Wire Line
+	15750 5950 15750 5850
+Wire Wire Line
+	15750 5850 16150 5850
 $EndSCHEMATC

Commit message: Added v3 garden controller hardware
Parts:
- removed C10, C2, C22: 0.1uF, Capacitor_SMD:C_0402_1005Metric, symbol Device:C
- removed C17: 33pF, Capacitor_SMD:C_0402_1005Metric, symbol Device:C
- removed C23, C25, C27: 0.1uF/50V, Capacitor_SMD:C_0603_1608Metric, symbol Device:C
- removed C24, C26, C28: 1uF/50V, Capacitor_SMD:C_0805_2012Metric, symbol Device:C
- removed C3: 1uF, Capacitor_SMD:C_0402_1005Metric, symbol Device:C
- removed C7: 22uF, Capacitor_SMD:C_0805_2012Metric, symbol Device:C
- removed C8: 10uF, Capacitor_SMD:C_0402_1005Metric, symbol Device:C
- removed D10: D, Diode_SMD:D_SOD-323F, symbol Device:D
- removed D3: GREEN, LED_SMD:LED_0603_1608Metric, symbol ostrich-rescue:LED-device
- removed J10: CONN_01X09, TerminalBlock_Phoenix:TerminalBlock_Phoenix_MKDS-3-9-5.08_1x09_P5.08mm_Horizontal, symbol conn1:CONN_01X09
- removed J9: USB_B_Micro, Connector_USB:USB_Micro-B_Molex-105017-0001, symbol Connector:USB_B_Micro
- removed JP1: Jumper, Jumper:SolderJumper-2_P1.3mm_Open_RoundedPad1.0x1.5mm, symbol Device:Jumper
- removed M2, M3, M4, M5: CONN_01X01, MountingHole:MountingHole_6.4mm_M6, symbol conn1:CONN_01X01
- removed R24, R28: 10kR, Resistor_SMD:R_0402_1005Metric, symbol Device:R
- removed R7: 100R, Resistor_SMD:R_0402_1005Metric, symbol ostrich-rescue:R-device
- removed TP1, TP10, TP11, TP12, TP13, TP2, TP3, TP4, TP5, TP6, TP7, TP8, TP9: TestPoint, TestPoint:TestPoint_Loop_D3.50mm_Drill1.4mm_Beaded, symbol Connector:TestPoint
- removed U10: DHT11, Sensor:Aosong_DHT11_5.5x12.0_P2.54mm, symbol Sensor:DHT11
- removed U11: AZ1117-3.3, Package_TO_SOT_THT:TO-220-3_Vertical, symbol Regulator_Linear:AZ1117-3.3
- removed U12, U13, U14: MCP1416, Package_TO_SOT_SMD:SOT-23-5, symbol Driver_FET:MCP1416
- removed U3: CP2102, Package_DFN_QFN:QFN-28-1EP_5x5mm_P0.5mm_EP3.35x3.35mm, symbol Interface_USB:CP2102N-A01-GQFN28
- removed U5: INA226, Package_SO:VSSOP-10_3x3mm_P0.5mm, symbol Analog_ADC:INA226
- added C2: 220uF/25V, Capacitor_THT:CP_Radial_D8.0mm_P3.50mm, symbol Device:CP
- added D10, D12: D_Schottky, Diode_SMD:D_SOD-123, symbol Device:D_Schottky
- added D11, D3: D_Schottky, Diode_SMD:D_SOD-123, symbol garden-rescue:D_Schottky-device-ostrich-rescue
- added H1, H2, H3: MountingHole, MountingHole:MountingHole_3.2mm_M3, symbol Mechanical:MountingHole
- added J10: CONN_01X08, Connector_PinHeader_2.54mm:PinHeader_1x08_P2.54mm_Vertical, symbol conn1:CONN_01X08
- added J11, J12: CONN_01X02, TerminalBlock_Phoenix:TerminalBlock_Phoenix_MKDS-1,5-2-5.08_1x02_P5.08mm_Horizontal, symbol conn1:CONN_01X02
- added J9: USB_C_Receptacle_USB2.0, Connector_USB:USB_C_Receptacle_HRO_TYPE-C-31-M-12, symbol Connector:USB_C_Receptacle_USB2.0
- added JP1: SolderJumper_2_Open, Jumper:SolderJumper-2_P1.3mm_Open_TrianglePad1.0x1.5mm, symbol Jumper:SolderJumper_2_Open
- added Q6, Q7: AO3416, Package_TO_SOT_SMD:SOT-23, symbol Device:Q_NMOS_GSD
- added R7: 10kR, Resistor_SMD:R_0402_1005Metric, symbol Device:R
- added U3: CH340C, Package_SO:SOIC-16_3.9x9.9mm_P1.27mm, symbol Interface_USB:CH340C
- C15: value 22uF -> 10uF; LCSC C45783 -> C15850
- C21: value 10uF -> 22uF; footprint Capacitor_SMD:C_0402_1005Metric -> Capacitor_SMD:C_0603_1608Metric; LCSC C15525 -> C59461
- D1, D2: value D -> 1N4148
- D4, D5, D6: symbol ostrich-rescue:LED-device -> garden-rescue:LED-device-ostrich-rescue
- D7: footprint Diode_SMD:D_SMA -> Diode_SMD:D_SOD-123; LCSC C2480 -> C8598
- D8, D9: symbol ostrich-rescue:D_Schottky-device -> garden-rescue:D_Schottky-device-ostrich-rescue
- J2, J3, J4, J5, J6: footprint TerminalBlock_Phoenix:TerminalBlock_Phoenix_MKDS-3-2-5.08_1x02_P5.08mm_Horizontal -> TerminalBlock_Phoenix:TerminalBlock_Phoenix_MKDS-1,5-2-5.08_1x02_P5.08mm_Horizontal; LCSC (none) -> C480516
- Q2: value Q_NMOS_GDS -> AO3416; footprint Package_TO_SOT_SMD:TO-252-2 -> Package_TO_SOT_SMD:SOT-23; symbol Device:Q_NMOS_GDS -> Device:Q_NMOS_GSD; LCSC C145546 -> C43307
- Q3: value Q_NMOS_GDS -> AO3416; footprint Package_TO_SOT_SMD:TO-252-2 -> Package_TO_SOT_SMD:SOT-23; symbol Device:Q_NMOS_GDS -> Device:Q_NMOS_GSD
- Q5: value Q_NMOS_GDS -> Q_NMOS_GSD/60V; footprint Package_TO_SOT_SMD:TO-252-2 -> Package_TO_SOT_SMD:SOT-23; symbol Device:Q_NMOS_GDS -> Device:Q_NMOS_GSD; LCSC C145546 -> C282260
- R10, R8, R9: symbol ostrich-rescue:R-device -> garden-rescue:R-device-ostrich-rescue
- R13: value 2kR -> 5.1k; LCSC C4109 -> C25905
- R20: value 0.1R -> 10kR; footprint Resistor_SMD:R_1206_3216Metric -> Resistor_SMD:R_0402_1005Metric; LCSC C25334 -> C25744
- R22: value 124kR -> 49.9k; LCSC C36777 -> C25897
- R23: value 40.2kR -> 16.2k; footprint Resistor_SMD:R_0603_1608Metric -> Resistor_SMD:R_0402_1005Metric; LCSC C12447 -> C27176
- R3: value 1kR -> 5.1k; LCSC C11702 -> C25905
- U4: LCSC (none) -> C82899
- U9: value MP2451DT -> MP2359; footprint Package_TO_SOT_SMD:SOT-23-6 -> Package_TO_SOT_SMD:TSOT-23-6; LCSC C14123 -> C14259
Connections:
- net labels added: CC1, CC2, Dm, Dp, IO14, IO15, IO32, IO34, IO35, SW2, SW3, Vbus
- net labels removed: 3V3_SHUNT_N, 3V3_SHUNT_P, DHT22, I35, I36, I39, IO18, IO5, LED3, PRESSURE_SW_GATE, PRES_SHUNT_N, PRES_SHUNT_P, SW0_GATE, SW1_GATE
- wire segments 247 -> 271
- no-connect marks 2 -> 6
Other:
- note added: "Battery conn"
- note added: "Expansion Port"
- note added: "Ext I2C Bus"
- note added: "MCU"
- note added: "Mounting holes"
- note added: "Power Input"
- note added: "Pressure Transducer (24V/4-20mA current loop)"
- note added: "SmartSolar VE Direct"
- note added: "Solar charger conn"
- note added: "Switched Outputs"
- note removed: "Backup 3.3V LDO"
- note removed: "Battery (with pass-through monitoring for current integration)"
- note removed: "FET drivers"
- note removed: "Future Expansion"
- note removed: "I2C Sensors"
- note removed: "M6 mounting holes"
- note removed: "MCU + WiFi"
- note removed: "Pressure transducer (4-20mA current loop)"
- note removed: "SmartSolar VE Direct interface"
- note removed: "Switched outputs"
- note removed: "Temp/Humidity"
- moved on the sheet: D4, D5, D6, D8, D9, R10, R8, R9

Commit message: Updated garden and temp sensor hw
Parts:
- J11, J12, J2, J3, J4, J5, J6: LCSC C480516 -> C395868
- J7, J8: LCSC (none) -> C474922
- Q3, Q7: LCSC C145546 -> C43307
Changed lines of the file:
@@
 F 2 "TerminalBlock_Phoenix:TerminalBlock_Phoenix_MKDS-1,5-2-5.08_1x02_P5.08mm_Horizontal" H 1400 9050 50  0001 C CNN
 F 3 "" H 1400 9050 50  0001 C CNN
-F 4 "C480516" H 1400 9050 50  0001 C CNN "LCSC"
+F 4 "C395868" H 1400 9050 50  0001 C CNN "LCSC"
 	1    1400 9050
 	1    0    0    1
@@
 F 2 "Package_TO_SOT_SMD:SOT-23" H 10950 2200 50  0001 C CNN
 F 3 "~" H 10750 2100 50  0001 C CNN
-F 4 "C145546" H 10750 2100 50  0001 C CNN "LCSC"
+F 4 "C43307" H 10750 2100 50  0001 C CNN "LCSC"
 	1    10750 2100
 	1    0    0    -1
@@
 F 2 "TerminalBlock_Phoenix:TerminalBlock_Phoenix_MKDS-1,5-2-5.08_1x02_P5.08mm_Horizontal" H 9950 1700 50  0001 C CNN
 F 3 "" H 9950 1700 50  0001 C CNN
-F 4 "C480516" H 9950 1700 50  0001 C CNN "LCSC"
+F 4 "C395868" H 9950 1700 50  0001 C CNN "LCSC"
 	1    9950 1700
 	1    0    0    1
@@
 F 2 "TerminalBlock_Phoenix:TerminalBlock_Phoenix_MKDS-1,5-2-5.08_1x02_P5.08mm_Horizontal" H 11600 1750 50  0001 C CNN
 F 3 "" H 11600 1750 50  0001 C CNN
-F 4 "C480516" H 11600 1750 50  0001 C CNN "LCSC"
+F 4 "C395868" H 11600 1750 50  0001 C CNN "LCSC"
 	1    11600 1750
 	1    0    0    1
@@
 F 2 "TerminalBlock_Phoenix:TerminalBlock_Phoenix_MKDS-1,5-2-5.08_1x02_P5.08mm_Horizontal" H 7100 10000 50  0001 C CNN
 F 3 "" H 7100 10000 50  0001 C CNN
-F 4 "C480516" H 7100 10000 50  0001 C CNN "LCSC"
+F 4 "C395868" H 7100 10000 50  0001 C CNN "LCSC"
 	1    7100 10000
 	1    0    0    1
@@
 F 2 "TerminalBlock_Phoenix:TerminalBlock_Phoenix_MPT-0,5-4-2.54_1x04_P2.54mm_Horizontal" H 5650 8350 50  0001 C CNN
 F 3 "" H 5650 8350 50  0001 C CNN
+F 4 "C474922" H 5650 8350 50  0001 C CNN "LCSC"
 	1    5650 8350
 	1    0    0    -1
@@
 F 2 "TerminalBlock_Phoenix:TerminalBlock_Phoenix_MPT-0,5-4-2.54_1x04_P2.54mm_Horizontal" H 6450 8350 50  0001 C CNN
 F 3 "" H 6450 8350 50  0001 C CNN
+F 4 "C474922" H 6450 8350 50  0001 C CNN "LCSC"
 	1    6450 8350
 	1    0    0    -1
@@
 F 2 "TerminalBlock_Phoenix:TerminalBlock_Phoenix_MKDS-1,5-2-5.08_1x02_P5.08mm_Horizontal" H 2700 8450 50  0001 C CNN
 F 3 "" H 2700 8450 50  0001 C CNN
-F 4 "C480516" H 2700 8450 50  0001 C CNN "LCSC"
+F 4 "C395868" H 2700 8450 50  0001 C CNN "LCSC"
 	1    2700 8450
 	1    0    0    1
@@
 F 2 "Package_TO_SOT_SMD:SOT-23" H 10900 3600 50  0001 C CNN
 F 3 "~" H 10700 3500 50  0001 C CNN
-F 4 "C145546" H 10700 3500 50  0001 C CNN "LCSC"
+F 4 "C43307" H 10700 3500 50  0001 C CNN "LCSC"
 	1    10700 3500
 	1    0    0    -1
@@
 F 2 "TerminalBlock_Phoenix:TerminalBlock_Phoenix_MKDS-1,5-2-5.08_1x02_P5.08mm_Horizontal" H 9900 3100 50  0001 C CNN
 F 3 "" H 9900 3100 50  0001 C CNN
-F 4 "C480516" H 9900 3100 50  0001 C CNN "LCSC"
+F 4 "C395868" H 9900 3100 50  0001 C CNN "LCSC"
 	1    9900 3100
 	1    0    0    1
@@
 F 2 "TerminalBlock_Phoenix:TerminalBlock_Phoenix_MKDS-1,5-2-5.08_1x02_P5.08mm_Horizontal" H 11550 3150 50  0001 C CNN
 F 3 "" H 11550 3150 50  0001 C CNN
-F 4 "C480516" H 11550 3150 50  0001 C CNN "LCSC"
+F 4 "C395868" H 11550 3150 50  0001 C CNN "LCSC"
 	1    11550 3150
 	1    0    0    1

Commit message: Updated garden controller hardware to version 4
Parts:
- removed C11: 0.1uF/50V, Capacitor_SMD:C_0603_1608Metric, symbol Device:C
- removed C12, C13: 1uF/50V, Capacitor_SMD:C_0805_2012Metric, symbol Device:C
- removed C14: 10uF/50V, Capacitor_SMD:C_1206_3216Metric, symbol Device:C
- removed D1, D2: 1N4148, Diode_SMD:D_SOD-323F, symbol Device:D
- removed JP1: SolderJumper_2_Open, Jumper:SolderJumper-2_P1.3mm_Open_TrianglePad1.0x1.5mm, symbol Jumper:SolderJumper_2_Open
- removed R31: 10kR, Resistor_SMD:R_0402_1005Metric, symbol Device:R
- removed U1, U2: INA226, Package_SO:VSSOP-10_3x3mm_P0.5mm, symbol Analog_ADC:INA226
- removed U4: ESP32-WROOM-32, RF_Module:ESP32-WROOM-32, symbol RF_Module:ESP32-WROOM-32
- removed U7: MCP1416, Package_TO_SOT_SMD:SOT-23-5, symbol Driver_FET:MCP1416
- added AE1: Antenna_Dipole, Antennas:TI_DN007_2.4GHz, symbol Device:Antenna_Dipole
- added C10: 22uF, Capacitor_SMD:C_0603_1608Metric, symbol Device:C
- added C3, C5, C8: 0.1uF, Capacitor_SMD:C_0402_1005Metric, symbol Device:C
- added C7: DNP, Capacitor_SMD:C_0402_1005Metric, symbol Device:C
- added D13, D14: D_Schottky, Diode_SMD:D_SOD-123, symbol garden-rescue:D_Schottky-device-ostrich-rescue
- added J13: CONN_01X02, modular_blocks:KF2EDGR-3.5-2P, symbol conn1:CONN_01X02
- added J14, J16: CONN_01X03, Connector_JST:JST_PH_S3B-PH-SM4-TB_1x03-1MP_P2.00mm_Horizontal, symbol conn1:CONN_01X03
- added LOGO1: LOGO, Logos:qwiic, symbol qwiic:LOGO
- added LOGO2: Logo_Open_Hardware_Large, Symbol:OSHW-Logo2_9.8x8mm_SilkScreen, symbol Graphic:Logo_Open_Hardware_Large
- added Q10, Q9: YJL3416A, Package_TO_SOT_SMD:SOT-23, symbol Device:Q_NMOS_GSD
- added Q8: Q_PMOS_GDS, Package_TO_SOT_SMD:SOT-23, symbol Device:Q_PMOS_GSD
- added R24: 1kR, Resistor_SMD:R_0402_1005Metric, symbol Device:R
- added R28: 100kR, Resistor_SMD:R_0402_1005Metric, symbol Device:R
- added R29, R30: 10kR, Resistor_SMD:R_0402_1005Metric, symbol Device:R
- added U1: SHT30-DIS, Sensor_Humidity:Sensirion_DFN-8-1EP_2.5x2.5mm_P0.5mm_EP1.1x1.7mm, symbol Sensor_Humidity:SHT30-DIS
- added U2: INA3221, Package_DFN_QFN:Texas_RGV_S-PVQFN-N16_EP2.1x2.1mm, symbol Power_Management:INA3221
- added U6: ESP32-PICO-V3, Package_DFN_QFN:QFN-48-1EP_7x7mm_P0.5mm_EP5.3x5.3mm, symbol esp32:ESP32-PICO-V3
- C1: value 0.1uF -> DNP; LCSC C1525 -> (none)
- J1: footprint Connector_JST:JST_PH_B4B-PH-SM4-TB_1x04-1MP_P2.00mm_Vertical -> Connector_JST:JST_PH_S4B-PH-K_1x04_P2.00mm_Horizontal; LCSC (none) -> C157926
- J10: value CONN_01X08 -> CONN_01X06; footprint Connector_PinHeader_2.54mm:PinHeader_1x08_P2.54mm_Vertical -> Connector_PinHeader_2.54mm:PinHeader_1x06_P2.54mm_Vertical; symbol conn1:CONN_01X08 -> conn1:CONN_01X06
- J11, J12, J3, J4, J5, J6: footprint TerminalBlock_Phoenix:TerminalBlock_Phoenix_MKDS-1,5-2-5.08_1x02_P5.08mm_Horizontal -> modular_blocks:KF2EDGR-3.5-2P; LCSC C395868 -> C441171
- J2: footprint TerminalBlock_Phoenix:TerminalBlock_Phoenix_MKDS-1,5-2-5.08_1x02_P5.08mm_Horizontal -> modular_blocks:WJ2EDGRC-5-08-2P; LCSC C395868 -> C3697
- J7: footprint TerminalBlock_Phoenix:TerminalBlock_Phoenix_MPT-0,5-4-2.54_1x04_P2.54mm_Horizontal -> Connector_JST:JST_SH_SM04B-SRSS-TB_1x04-1MP_P1.00mm_Horizontal; LCSC C474922 -> C437064
- J8: footprint TerminalBlock_Phoenix:TerminalBlock_Phoenix_MPT-0,5-4-2.54_1x04_P2.54mm_Horizontal -> modular_blocks:KF2EDGR-3.5-4P; LCSC C474922 -> C441173
- L1: value 4.7uH -> 3.3uH; footprint MWSA0603:MWSA0603 -> Inductors:SWPA30xxS; LCSC C132139 -> C48020
- Q2, Q3, Q6, Q7: value AO3416 -> YJL3416A; LCSC C43307 -> C389061
- R2: value 12mR -> 5mR; LCSC C76243 -> C371096
- R27: value 10kR -> 100kR; LCSC C25744 -> C25741
- R4: value 2.2kR -> 0R; LCSC C25879 -> C17168
- R6: value 2.2R -> 6.8R; footprint Resistor_SMD:R_0603_1608Metric -> Resistor_SMD:R_0402_1005Metric; LCSC C22939 -> C409930
- U9: value MP2359 -> TPMP2359; LCSC C14259 -> C2959845
Connections:
- net labels added: CC1_ADC, CC2_ADC, GRAVITY0, GRAVITY1, LNA, PRES_SHUNT_N, PRES_SHUNT_P, SW4, SW5, Vbus_blocked, ~Vbus_to_12V_EN
- net labels removed: ALERT, IO14, IO15, IO32, IO34, IO35, PRESSURE_PWR
- wire segments 271 -> 273
Other:
- note added: "0.005R * 32A = 163mV"
- note added: "6.8R * 24mA = 163mV"
- note added: "Current Monitors"
- note added: "Gravity Ports"
- note added: "Grounded Coplanar Wave Guide (JLC7628 Substrate):\nCalculator: https://spok.ca/index.php/resources/tools/99-cpwcalc\nH = 0.18, W=0.295, T=0.035, S=0.2, Er=4.6, Z0 = 50.05R\n\n1mm PCB"
- note added: "Open Source Hardware"
- note added: "Pressure Transducer (12V/4-20mA current loop)"
- note added: "RF"
- note added: "Shunt full scale: 163.8mV"
- note added: "Temperature + Humidity"
- note removed: "Expansion Port"
- note removed: "Pressure Transducer (24V/4-20mA current loop)"
- note removed: "Solar charger conn"
- moved on the sheet: D11, D3, D8, D9
