File: hardware/light_control/light_control/light_control.kicad_pcb (KiCad board)
At the start: 4 copper layers, 59.7 x 48.3 mm, 69 parts, among them J1 Screw_Terminal_01x02, J10 Screw_Terminal_01x02, J11 Screw_Terminal_01x02, J12 Conn_01x03, J2 USB_B_Micro, J3 Screw_Terminal_01x02, J4 Screw_Terminal_01x02, J5 Screw_Terminal_01x02, J6 Screw_Terminal_01x02, J7 Screw_Terminal_01x02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

Commit message: Updated hardware
Parts:
- added R17: 10kR, Resistor_SMD:R_0402_1005Metric, F.Cu at (121.2, 86.4)
- added R18: 10kR, Resistor_SMD:R_0402_1005Metric, F.Cu at (136.3, 88.1)
- added R19: 10kR, Resistor_SMD:R_0402_1005Metric, F.Cu at (144.4, 83.4)
- added R20: 10kR, Resistor_SMD:R_0402_1005Metric, F.Cu at (145.9, 77.5)
- added R21: 10kR, Resistor_SMD:R_0402_1005Metric, F.Cu at (127.4, 88.3)
- added R22: 10kR, Resistor_SMD:R_0402_1005Metric, F.Cu at (142.7, 86.9)
- added R23: 10kR, Resistor_SMD:R_0402_1005Metric, F.Cu at (144.4, 82.0)
- added R24: 10kR, Resistor_SMD:R_0402_1005Metric, F.Cu at (147.3, 68.9)
- Q3: value Q_NMOS_GDS -> Q_NMOS_GSD
- moved R8 1.89 mm to (129.3, 88.3), turned to 180 degrees
- moved R4 1.69 mm to (122.7, 86.6), turned to 90 degrees
- moved Q5 1.27 mm to (148.6, 89.9), turned to 270 degrees
- moved R10 0.65 mm to (147.4, 82.5), turned to 270 degrees
- moved Q8 0.27 mm to (141.9, 89.7), turned to 270 degrees
- moved Q3 0.21 mm to (121.8, 89.4), turned to 270 degrees
- moved Q7 0.18 mm to (128.2, 90.7), turned to 270 degrees
- turned Q10 to 0 degrees
- turned Q4 to 270 degrees
- turned Q6 to 0 degrees
- turned Q9 to 0 degrees
- turned R11 to 270 degrees
Connections:
- Q10 pad 2: Net-(D10-Pad2) -> GND
- Q10 pad 3: GND -> Net-(D10-Pad2)
- Q3 pad 2: Net-(D3-Pad2) -> GND
- Q3 pad 3: GND -> Net-(D3-Pad2)
- Q4 pad 2: Net-(D4-Pad2) -> GND
- Q4 pad 3: GND -> Net-(D4-Pad2)
- Q5 pad 2: Net-(D5-Pad2) -> GND
- Q5 pad 3: GND -> Net-(D5-Pad2)
- Q6 pad 2: Net-(D6-Pad2) -> GND
- Q6 pad 3: GND -> Net-(D6-Pad2)
- Q7 pad 2: Net-(D7-Pad2) -> GND
- Q7 pad 3: GND -> Net-(D7-Pad2)
- Q8 pad 2: Net-(D8-Pad2) -> GND
- Q8 pad 3: GND -> Net-(D8-Pad2)
- Q9 pad 2: Net-(D9-Pad2) -> GND
- Q9 pad 3: GND -> Net-(D9-Pad2)
Routing:
- net GND: track 65.1 -> 73.5 mm, vias 27 -> 34
- net Net-(D6-Pad2): track 7.33 -> 10.4 mm
- net Net-(Q5-Pad1): track 4.30 -> 6.76 mm
- net /CH_8: track 9.49 -> 11.4 mm
- net /CH_4: track 28.1 -> 29.7 mm
- net Net-(Q6-Pad1): track 1.53 -> 3.08 mm
- net /CH_5: track 17.9 -> 19.4 mm
- net Net-(Q8-Pad1): track 1.69 -> 2.95 mm
- net /CH_3: track 24.0 -> 25.1 mm
- net Net-(D3-Pad2): track 8.26 -> 9.31 mm
- net /LED4: track 18.0 -> 19.0 mm
- net Net-(D9-Pad2): track 6.85 -> 7.83 mm
- net Net-(Q4-Pad1): track 1.40 -> 2.37 mm
- net /CH_6: track 9.99 -> 10.9 mm
- net /CH_2: track 20.9 -> 21.6 mm
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Other:
- board text added: "Rev 2"
- board text removed: "Rev 1"
